File: LEDs.kicad_sch (KiCad schematic)
At the start: 160 parts

Commit message: auto layout of pcb including rgbw/caps
Parts:
- LED1: renamed from D84; footprint BOM:SK6812RGBW -> LED_SMD:LED_SK6812_PLCC4_5.0x5.0mm_P3.2mm; symbol LOCAL:SK6812RGBW-WS -> BOM:SK6812RGBW-WS
- LED10: renamed from D93; footprint BOM:SK6812RGBW -> LED_SMD:LED_SK6812_PLCC4_5.0x5.0mm_P3.2mm; symbol LOCAL:SK6812RGBW-WS -> BOM:SK6812RGBW-WS
- LED11: renamed from D94; footprint BOM:SK6812RGBW -> LED_SMD:LED_SK6812_PLCC4_5.0x5.0mm_P3.2mm; symbol LOCAL:SK6812RGBW-WS -> BOM:SK6812RGBW-WS
- LED12: renamed from D95; footprint BOM:SK6812RGBW -> LED_SMD:LED_SK6812_PLCC4_5.0x5.0mm_P3.2mm; symbol LOCAL:SK6812RGBW-WS -> BOM:SK6812RGBW-WS
- LED13: renamed from D96; footprint BOM:SK6812RGBW -> LED_SMD:LED_SK6812_PLCC4_5.0x5.0mm_P3.2mm; symbol LOCAL:SK6812RGBW-WS -> BOM:SK6812RGBW-WS
- LED14: renamed from D97; footprint BOM:SK6812RGBW -> LED_SMD:LED_SK6812_PLCC4_5.0x5.0mm_P3.2mm; symbol LOCAL:SK6812RGBW-WS -> BOM:SK6812RGBW-WS
- LED15: renamed from D98; footprint BOM:SK6812RGBW -> LED_SMD:LED_SK6812_PLCC4_5.0x5.0mm_P3.2mm; symbol LOCAL:SK6812RGBW-WS -> BOM:SK6812RGBW-WS
- LED16: renamed from D99; footprint BOM:SK6812RGBW -> LED_SMD:LED_SK6812_PLCC4_5.0x5.0mm_P3.2mm; symbol LOCAL:SK6812RGBW-WS -> BOM:SK6812RGBW-WS
- LED17: renamed from D100; footprint BOM:SK6812RGBW -> LED_SMD:LED_SK6812_PLCC4_5.0x5.0mm_P3.2mm; symbol LOCAL:SK6812RGBW-WS -> BOM:SK6812RGBW-WS
- LED18: renamed from D101; footprint BOM:SK6812RGBW -> LED_SMD:LED_SK6812_PLCC4_5.0x5.0mm_P3.2mm; symbol LOCAL:SK6812RGBW-WS -> BOM:SK6812RGBW-WS
- LED19: renamed from D102; footprint BOM:SK6812RGBW -> LED_SMD:LED_SK6812_PLCC4_5.0x5.0mm_P3.2mm; symbol LOCAL:SK6812RGBW-WS -> BOM:SK6812RGBW-WS
- LED2: renamed from D85; footprint BOM:SK6812RGBW -> LED_SMD:LED_SK6812_PLCC4_5.0x5.0mm_P3.2mm; symbol LOCAL:SK6812RGBW-WS -> BOM:SK6812RGBW-WS
- LED20: renamed from D103; footprint BOM:SK6812RGBW -> LED_SMD:LED_SK6812_PLCC4_5.0x5.0mm_P3.2mm; symbol LOCAL:SK6812RGBW-WS -> BOM:SK6812RGBW-WS
- LED21: renamed from D104; footprint BOM:SK6812RGBW -> LED_SMD:LED_SK6812_PLCC4_5.0x5.0mm_P3.2mm; symbol LOCAL:SK6812RGBW-WS -> BOM:SK6812RGBW-WS
- LED22: renamed from D105; footprint BOM:SK6812RGBW -> LED_SMD:LED_SK6812_PLCC4_5.0x5.0mm_P3.2mm; symbol LOCAL:SK6812RGBW-WS -> BOM:SK6812RGBW-WS
- LED23: renamed from D106; footprint BOM:SK6812RGBW -> LED_SMD:LED_SK6812_PLCC4_5.0x5.0mm_P3.2mm; symbol LOCAL:SK6812RGBW-WS -> BOM:SK6812RGBW-WS
- LED24: renamed from D107; footprint BOM:SK6812RGBW -> LED_SMD:LED_SK6812_PLCC4_5.0x5.0mm_P3.2mm; symbol LOCAL:SK6812RGBW-WS -> BOM:SK6812RGBW-WS
- LED25: renamed from D108; footprint BOM:SK6812RGBW -> LED_SMD:LED_SK6812_PLCC4_5.0x5.0mm_P3.2mm; symbol LOCAL:SK6812RGBW-WS -> BOM:SK6812RGBW-WS
- LED26: renamed from D109; footprint BOM:SK6812RGBW -> LED_SMD:LED_SK6812_PLCC4_5.0x5.0mm_P3.2mm; symbol LOCAL:SK6812RGBW-WS -> BOM:SK6812RGBW-WS
- LED27: renamed from D110; footprint BOM:SK6812RGBW -> LED_SMD:LED_SK6812_PLCC4_5.0x5.0mm_P3.2mm; symbol LOCAL:SK6812RGBW-WS -> BOM:SK6812RGBW-WS
- LED28: renamed from D111; footprint BOM:SK6812RGBW -> LED_SMD:LED_SK6812_PLCC4_5.0x5.0mm_P3.2mm; symbol LOCAL:SK6812RGBW-WS -> BOM:SK6812RGBW-WS
- LED29: renamed from D112; footprint BOM:SK6812RGBW -> LED_SMD:LED_SK6812_PLCC4_5.0x5.0mm_P3.2mm; symbol LOCAL:SK6812RGBW-WS -> BOM:SK6812RGBW-WS
- LED3: renamed from D86; footprint BOM:SK6812RGBW -> LED_SMD:LED_SK6812_PLCC4_5.0x5.0mm_P3.2mm; symbol LOCAL:SK6812RGBW-WS -> BOM:SK6812RGBW-WS
- LED30: renamed from D113; footprint BOM:SK6812RGBW -> LED_SMD:LED_SK6812_PLCC4_5.0x5.0mm_P3.2mm; symbol LOCAL:SK6812RGBW-WS -> BOM:SK6812RGBW-WS
- LED31: renamed from D114; footprint BOM:SK6812RGBW -> LED_SMD:LED_SK6812_PLCC4_5.0x5.0mm_P3.2mm; symbol LOCAL:SK6812RGBW-WS -> BOM:SK6812RGBW-WS
- LED32: renamed from D115; footprint BOM:SK6812RGBW -> LED_SMD:LED_SK6812_PLCC4_5.0x5.0mm_P3.2mm; symbol LOCAL:SK6812RGBW-WS -> BOM:SK6812RGBW-WS
- LED33: renamed from D116; footprint BOM:SK6812RGBW -> LED_SMD:LED_SK6812_PLCC4_5.0x5.0mm_P3.2mm; symbol LOCAL:SK6812RGBW-WS -> BOM:SK6812RGBW-WS
- LED34: renamed from D117; footprint BOM:SK6812RGBW -> LED_SMD:LED_SK6812_PLCC4_5.0x5.0mm_P3.2mm; symbol LOCAL:SK6812RGBW-WS -> BOM:SK6812RGBW-WS
- LED35: renamed from D118; footprint BOM:SK6812RGBW -> LED_SMD:LED_SK6812_PLCC4_5.0x5.0mm_P3.2mm; symbol LOCAL:SK6812RGBW-WS -> BOM:SK6812RGBW-WS
- LED36: renamed from D119; footprint BOM:SK6812RGBW -> LED_SMD:LED_SK6812_PLCC4_5.0x5.0mm_P3.2mm; symbol LOCAL:SK6812RGBW-WS -> BOM:SK6812RGBW-WS
- LED37: renamed from D120; footprint BOM:SK6812RGBW -> LED_SMD:LED_SK6812_PLCC4_5.0x5.0mm_P3.2mm; symbol LOCAL:SK6812RGBW-WS -> BOM:SK6812RGBW-WS
- LED38: renamed from D121; footprint BOM:SK6812RGBW -> LED_SMD:LED_SK6812_PLCC4_5.0x5.0mm_P3.2mm; symbol LOCAL:SK6812RGBW-WS -> BOM:SK6812RGBW-WS
- LED39: renamed from D122; footprint BOM:SK6812RGBW -> LED_SMD:LED_SK6812_PLCC4_5.0x5.0mm_P3.2mm; symbol LOCAL:SK6812RGBW-WS -> BOM:SK6812RGBW-WS
- LED4: renamed from D87; footprint BOM:SK6812RGBW -> LED_SMD:LED_SK6812_PLCC4_5.0x5.0mm_P3.2mm; symbol LOCAL:SK6812RGBW-WS -> BOM:SK6812RGBW-WS
- LED40: renamed from D123; footprint BOM:SK6812RGBW -> LED_SMD:LED_SK6812_PLCC4_5.0x5.0mm_P3.2mm; symbol LOCAL:SK6812RGBW-WS -> BOM:SK6812RGBW-WS
- LED41: renamed from D124; footprint BOM:SK6812RGBW -> LED_SMD:LED_SK6812_PLCC4_5.0x5.0mm_P3.2mm; symbol LOCAL:SK6812RGBW-WS -> BOM:SK6812RGBW-WS
- LED42: renamed from D125; footprint BOM:SK6812RGBW -> LED_SMD:LED_SK6812_PLCC4_5.0x5.0mm_P3.2mm; symbol LOCAL:SK6812RGBW-WS -> BOM:SK6812RGBW-WS
- LED43: renamed from D126; footprint BOM:SK6812RGBW -> LED_SMD:LED_SK6812_PLCC4_5.0x5.0mm_P3.2mm; symbol LOCAL:SK6812RGBW-WS -> BOM:SK6812RGBW-WS
- LED44: renamed from D127; footprint BOM:SK6812RGBW -> LED_SMD:LED_SK6812_PLCC4_5.0x5.0mm_P3.2mm; symbol LOCAL:SK6812RGBW-WS -> BOM:SK6812RGBW-WS
- LED45: renamed from D128; footprint BOM:SK6812RGBW -> LED_SMD:LED_SK6812_PLCC4_5.0x5.0mm_P3.2mm; symbol LOCAL:SK6812RGBW-WS -> BOM:SK6812RGBW-WS
- LED46: renamed from D129; footprint BOM:SK6812RGBW -> LED_SMD:LED_SK6812_PLCC4_5.0x5.0mm_P3.2mm; symbol LOCAL:SK6812RGBW-WS -> BOM:SK6812RGBW-WS
- LED47: renamed from D130; footprint BOM:SK6812RGBW -> LED_SMD:LED_SK6812_PLCC4_5.0x5.0mm_P3.2mm; symbol LOCAL:SK6812RGBW-WS -> BOM:SK6812RGBW-WS
- LED48: renamed from D131; footprint BOM:SK6812RGBW -> LED_SMD:LED_SK6812_PLCC4_5.0x5.0mm_P3.2mm; symbol LOCAL:SK6812RGBW-WS -> BOM:SK6812RGBW-WS
- LED49: renamed from D132; footprint BOM:SK6812RGBW -> LED_SMD:LED_SK6812_PLCC4_5.0x5.0mm_P3.2mm; symbol LOCAL:SK6812RGBW-WS -> BOM:SK6812RGBW-WS
- LED5: renamed from D88; footprint BOM:SK6812RGBW -> LED_SMD:LED_SK6812_PLCC4_5.0x5.0mm_P3.2mm; symbol LOCAL:SK6812RGBW-WS -> BOM:SK6812RGBW-WS
- LED50: renamed from D133; footprint BOM:SK6812RGBW -> LED_SMD:LED_SK6812_PLCC4_5.0x5.0mm_P3.2mm; symbol LOCAL:SK6812RGBW-WS -> BOM:SK6812RGBW-WS
- LED51: renamed from D134; footprint BOM:SK6812RGBW -> LED_SMD:LED_SK6812_PLCC4_5.0x5.0mm_P3.2mm; symbol LOCAL:SK6812RGBW-WS -> BOM:SK6812RGBW-WS
- LED52: renamed from D135; footprint BOM:SK6812RGBW -> LED_SMD:LED_SK6812_PLCC4_5.0x5.0mm_P3.2mm; symbol LOCAL:SK6812RGBW-WS -> BOM:SK6812RGBW-WS
- LED53: renamed from D136; footprint BOM:SK6812RGBW -> LED_SMD:LED_SK6812_PLCC4_5.0x5.0mm_P3.2mm; symbol LOCAL:SK6812RGBW-WS -> BOM:SK6812RGBW-WS
- LED54: renamed from D137; footprint BOM:SK6812RGBW -> LED_SMD:LED_SK6812_PLCC4_5.0x5.0mm_P3.2mm; symbol LOCAL:SK6812RGBW-WS -> BOM:SK6812RGBW-WS
- LED55: renamed from D138; footprint BOM:SK6812RGBW -> LED_SMD:LED_SK6812_PLCC4_5.0x5.0mm_P3.2mm; symbol LOCAL:SK6812RGBW-WS -> BOM:SK6812RGBW-WS
- LED56: renamed from D139; footprint BOM:SK6812RGBW -> LED_SMD:LED_SK6812_PLCC4_5.0x5.0mm_P3.2mm; symbol LOCAL:SK6812RGBW-WS -> BOM:SK6812RGBW-WS
- LED57: renamed from D140; footprint BOM:SK6812RGBW -> LED_SMD:LED_SK6812_PLCC4_5.0x5.0mm_P3.2mm; symbol LOCAL:SK6812RGBW-WS -> BOM:SK6812RGBW-WS
- LED58: renamed from D141; footprint BOM:SK6812RGBW -> LED_SMD:LED_SK6812_PLCC4_5.0x5.0mm_P3.2mm; symbol LOCAL:SK6812RGBW-WS -> BOM:SK6812RGBW-WS
- LED59: renamed from D142; footprint BOM:SK6812RGBW -> LED_SMD:LED_SK6812_PLCC4_5.0x5.0mm_P3.2mm; symbol LOCAL:SK6812RGBW-WS -> BOM:SK6812RGBW-WS
- LED6: renamed from D89; footprint BOM:SK6812RGBW -> LED_SMD:LED_SK6812_PLCC4_5.0x5.0mm_P3.2mm; symbol LOCAL:SK6812RGBW-WS -> BOM:SK6812RGBW-WS
- LED60: renamed from D143; footprint BOM:SK6812RGBW -> LED_SMD:LED_SK6812_PLCC4_5.0x5.0mm_P3.2mm; symbol LOCAL:SK6812RGBW-WS -> BOM:SK6812RGBW-WS
- LED61: renamed from D144; footprint BOM:SK6812RGBW -> LED_SMD:LED_SK6812_PLCC4_5.0x5.0mm_P3.2mm; symbol LOCAL:SK6812RGBW-WS -> BOM:SK6812RGBW-WS
- LED62: renamed from D145; footprint BOM:SK6812RGBW -> LED_SMD:LED_SK6812_PLCC4_5.0x5.0mm_P3.2mm; symbol LOCAL:SK6812RGBW-WS -> BOM:SK6812RGBW-WS
- LED63: renamed from D146; footprint BOM:SK6812RGBW -> LED_SMD:LED_SK6812_PLCC4_5.0x5.0mm_P3.2mm; symbol LOCAL:SK6812RGBW-WS -> BOM:SK6812RGBW-WS
- LED64: renamed from D147; footprint BOM:SK6812RGBW -> LED_SMD:LED_SK6812_PLCC4_5.0x5.0mm_P3.2mm; symbol LOCAL:SK6812RGBW-WS -> BOM:SK6812RGBW-WS
- LED65: renamed from D148; footprint BOM:SK6812RGBW -> LED_SMD:LED_SK6812_PLCC4_5.0x5.0mm_P3.2mm; symbol LOCAL:SK6812RGBW-WS -> BOM:SK6812RGBW-WS
- LED66: renamed from D149; footprint BOM:SK6812RGBW -> LED_SMD:LED_SK6812_PLCC4_5.0x5.0mm_P3.2mm; symbol LOCAL:SK6812RGBW-WS -> BOM:SK6812RGBW-WS
- LED67: renamed from D150; footprint BOM:SK6812RGBW -> LED_SMD:LED_SK6812_PLCC4_5.0x5.0mm_P3.2mm; symbol LOCAL:SK6812RGBW-WS -> BOM:SK6812RGBW-WS
- LED68: renamed from D151; footprint BOM:SK6812RGBW -> LED_SMD:LED_SK6812_PLCC4_5.0x5.0mm_P3.2mm; symbol LOCAL:SK6812RGBW-WS -> BOM:SK6812RGBW-WS
- LED69: renamed from D152; footprint BOM:SK6812RGBW -> LED_SMD:LED_SK6812_PLCC4_5.0x5.0mm_P3.2mm; symbol LOCAL:SK6812RGBW-WS -> BOM:SK6812RGBW-WS
- LED7: renamed from D90; footprint BOM:SK6812RGBW -> LED_SMD:LED_SK6812_PLCC4_5.0x5.0mm_P3.2mm; symbol LOCAL:SK6812RGBW-WS -> BOM:SK6812RGBW-WS
- LED70: renamed from D153; footprint BOM:SK6812RGBW -> LED_SMD:LED_SK6812_PLCC4_5.0x5.0mm_P3.2mm; symbol LOCAL:SK6812RGBW-WS -> BOM:SK6812RGBW-WS
- LED71: renamed from D154; footprint BOM:SK6812RGBW -> LED_SMD:LED_SK6812_PLCC4_5.0x5.0mm_P3.2mm; symbol LOCAL:SK6812RGBW-WS -> BOM:SK6812RGBW-WS
- LED72: renamed from D155; footprint BOM:SK6812RGBW -> LED_SMD:LED_SK6812_PLCC4_5.0x5.0mm_P3.2mm; symbol LOCAL:SK6812RGBW-WS -> BOM:SK6812RGBW-WS
- LED73: renamed from D156; footprint BOM:SK6812RGBW -> LED_SMD:LED_SK6812_PLCC4_5.0x5.0mm_P3.2mm; symbol LOCAL:SK6812RGBW-WS -> BOM:SK6812RGBW-WS
- LED74: renamed from D157; footprint BOM:SK6812RGBW -> LED_SMD:LED_SK6812_PLCC4_5.0x5.0mm_P3.2mm; symbol LOCAL:SK6812RGBW-WS -> BOM:SK6812RGBW-WS
- LED75: renamed from D158; footprint BOM:SK6812RGBW -> LED_SMD:LED_SK6812_PLCC4_5.0x5.0mm_P3.2mm; symbol LOCAL:SK6812RGBW-WS -> BOM:SK6812RGBW-WS
- LED76: renamed from D159; footprint BOM:SK6812RGBW -> LED_SMD:LED_SK6812_PLCC4_5.0x5.0mm_P3.2mm; symbol LOCAL:SK6812RGBW-WS -> BOM:SK6812RGBW-WS
- LED77: renamed from D160; footprint BOM:SK6812RGBW -> LED_SMD:LED_SK6812_PLCC4_5.0x5.0mm_P3.2mm; symbol LOCAL:SK6812RGBW-WS -> BOM:SK6812RGBW-WS
- LED78: renamed from D161; footprint BOM:SK6812RGBW -> LED_SMD:LED_SK6812_PLCC4_5.0x5.0mm_P3.2mm; symbol LOCAL:SK6812RGBW-WS -> BOM:SK6812RGBW-WS
- LED79: renamed from D162; footprint BOM:SK6812RGBW -> LED_SMD:LED_SK6812_PLCC4_5.0x5.0mm_P3.2mm; symbol LOCAL:SK6812RGBW-WS -> BOM:SK6812RGBW-WS
- LED8: renamed from D91; footprint BOM:SK6812RGBW -> LED_SMD:LED_SK6812_PLCC4_5.0x5.0mm_P3.2mm; symbol LOCAL:SK6812RGBW-WS -> BOM:SK6812RGBW-WS
- LED80: renamed from D163; footprint BOM:SK6812RGBW -> LED_SMD:LED_SK6812_PLCC4_5.0x5.0mm_P3.2mm; symbol LOCAL:SK6812RGBW-WS -> BOM:SK6812RGBW-WS
- LED9: renamed from D92; footprint BOM:SK6812RGBW -> LED_SMD:LED_SK6812_PLCC4_5.0x5.0mm_P3.2mm; symbol LOCAL:SK6812RGBW-WS -> BOM:SK6812RGBW-WS
- renumbered C84 to C1, C93 to C10, C94 to C11, C95 to C12, C96 to C13, C97 to C14, C98 to C15, C99 to C16, C100 to C17, C101 to C18, C102 to C19, C85 to C2, C103 to C20, C104 to C21, C105 to C22, C106 to C23, C107 to C24, C108 to C25, C109 to C26, C110 to C27, C111 to C28, C112 to C29, C86 to C3, C113 to C30, C114 to C31, C115 to C32, C116 to C33, C117 to C34, C118 to C35, C119 to C36, C120 to C37, C121 to C38, C122 to C39, C87 to C4, C123 to C40, C124 to C41, C125 to C42, C126 to C43, C127 to C44, C128 to C45, C129 to C46, C130 to C47, C131 to C48, C132 to C49, C88 to C5, C133 to C50, C134 to C51, C135 to C52, C136 to C53, C137 to C54, C138 to C55, C139 to C56, C140 to C57, C141 to C58, C142 to C59, C89 to C6, C143 to C60, C144 to C61, C145 to C62, C146 to C63, C147 to C64, C148 to C65, C149 to C66, C150 to C67, C151 to C68, C152 to C69, C90 to C7, C153 to C70, C154 to C71, C155 to C72, C156 to C73, C157 to C74, C158 to C75, C159 to C76, C160 to C77, C161 to C78, C162 to C79, C91 to C8, C163 to C80, C92 to C9
Connections:
- net RGBW_DATA: now also LED13.2 (DIN); no longer LED1.2 (DIN)
- net at LED40.2 (DIN): now also LED41.4 (DOUT); no longer LED39.4 (DOUT)
- net at LED40.4 (DOUT): now also LED39.2 (DIN); no longer LED41.2 (DIN)
- net at LED32.2 (DIN): now also LED33.4 (DOUT); no longer LED31.4 (DOUT)
- net at LED32.4 (DOUT): now also LED31.2 (DIN); no longer LED33.2 (DIN)
- net at LED17.2 (DIN): now also LED18.4 (DOUT); no longer LED16.4 (DOUT)
- net at LED17.4 (DOUT): now also LED16.2 (DIN); no longer LED18.2 (DIN)
- net at LED63.2 (DIN): now also LED64.4 (DOUT); no longer LED62.4 (DOUT)
- net at LED63.4 (DOUT): now also LED62.2 (DIN); no longer LED64.2 (DIN)
- net at LED48.2 (DIN): now also LED49.4 (DOUT); no longer LED47.4 (DOUT)
- net at LED48.4 (DOUT): now also LED47.2 (DIN); no longer LED49.2 (DIN)
- net at LED7.2 (DIN): now also LED8.4 (DOUT); no longer LED6.4 (DOUT)
- net at LED7.4 (DOUT): now also LED6.2 (DIN); no longer LED8.2 (DIN)
- net at LED24.2 (DIN): now also LED25.4 (DOUT); no longer LED23.4 (DOUT)
- net at LED24.4 (DOUT): now also LED23.2 (DIN); no longer LED25.2 (DIN)
- net at LED19.2 (DIN): now also LED20.4 (DOUT); no longer LED18.4 (DOUT)
- net at LED76.2 (DIN): now also LED77.4 (DOUT); no longer LED75.4 (DOUT)
- net at LED76.4 (DOUT): now also LED75.2 (DIN); no longer LED77.2 (DIN)
- net at LED14.2 (DIN): now also LED15.4 (DOUT); no longer LED13.4 (DOUT)
- net at LED14.4 (DOUT): now also LED43.2 (DIN); no longer LED15.2 (DIN)
- net at LED35.2 (DIN): now also LED36.4 (DOUT); no longer LED34.4 (DOUT)
- net at LED35.4 (DOUT): now also LED34.2 (DIN); no longer LED36.2 (DIN)
- net at LED74.2 (DIN): now also LED75.4 (DOUT); no longer LED73.4 (DOUT)
- net at LED74.4 (DOUT): now also LED73.2 (DIN); no longer LED75.2 (DIN)
- net at LED53.2 (DIN): now also LED54.4 (DOUT); no longer LED52.4 (DOUT)
- net at LED53.4 (DOUT): now also LED52.2 (DIN); no longer LED54.2 (DIN)
- net at LED27.2 (DIN): now also LED28.4 (DOUT); no longer LED26.4 (DOUT)
- net at LED27.4 (DOUT): now also LED26.2 (DIN); no longer LED28.2 (DIN)
- net at LED72.4 (DOUT): no longer LED73.2 (DIN)
- net at LED38.4 (DOUT): now also LED37.2 (DIN); no longer LED39.2 (DIN)
- net at LED9.2 (DIN): now also LED10.4 (DOUT); no longer LED8.4 (DOUT)
- net at LED29.2 (DIN): now also LED30.4 (DOUT); no longer LED28.4 (DOUT)
- net at LED50.2 (DIN): now also LED51.4 (DOUT); no longer LED49.4 (DOUT)
- net at LED50.4 (DOUT): now also LED49.2 (DIN); no longer LED51.2 (DIN)
- net at LED5.2 (DIN): now also LED6.4 (DOUT); no longer LED4.4 (DOUT)
- net at LED5.4 (DOUT): now also LED4.2 (DIN); no longer LED6.2 (DIN)
- net at LED3.4 (DOUT): now also LED2.2 (DIN); no longer LED4.2 (DIN)
- net at LED38.2 (DIN): now also LED39.4 (DOUT); no longer LED37.4 (DOUT)
- net at LED55.2 (DIN): now also LED56.4 (DOUT); no longer LED54.4 (DOUT)
- net at LED19.4 (DOUT): now also LED18.2 (DIN); no longer LED20.2 (DIN)
- net at LED61.4 (DOUT): now also LED60.2 (DIN); no longer LED62.2 (DIN)
- net at LED78.2 (DIN): now also LED79.4 (DOUT); no longer LED77.4 (DOUT)
- net at LED69.2 (DIN): now also LED70.4 (DOUT); no longer LED68.4 (DOUT)
- net at LED69.4 (DOUT): now also LED68.2 (DIN); no longer LED70.2 (DIN)
- net at LED67.2 (DIN): now also LED68.4 (DOUT); no longer LED66.4 (DOUT)
- net at LED67.4 (DOUT): now also LED66.2 (DIN); no longer LED68.2 (DIN)
- net at LED71.2 (DIN): now also LED44.4 (DOUT); no longer LED70.4 (DOUT)
- net at LED72.2 (DIN): now also LED73.4 (DOUT); no longer LED71.4 (DOUT)
- net at LED44.2 (DIN): now also LED45.4 (DOUT); no longer LED43.4 (DOUT)
- net at LED45.2 (DIN): now also LED46.4 (DOUT); no longer LED44.4 (DOUT)
- net at LED1.4 (DOUT): now also LED28.2 (DIN); no longer LED2.2 (DIN)
- net at LED21.2 (DIN): now also LED22.4 (DOUT); no longer LED20.4 (DOUT)
- net at LED57.2 (DIN): now also LED29.4 (DOUT); no longer LED56.4 (DOUT)
- net at LED57.4 (DOUT): now also LED56.2 (DIN); no longer LED58.2 (DIN)
- net at LED65.4 (DOUT): now also LED64.2 (DIN); no longer LED66.2 (DIN)
- net at LED30.2 (DIN): now also LED31.4 (DOUT); no longer LED29.4 (DOUT)
- net at LED3.2 (DIN): now also LED4.4 (DOUT); no longer LED2.4 (DOUT)
- net at LED42.2 (DIN): now also LED43.4 (DOUT); no longer LED41.4 (DOUT)
- net at LED42.4 (DOUT): now also LED41.2 (DIN); no longer LED43.2 (DIN)
- net at LED61.2 (DIN): now also LED62.4 (DOUT); no longer LED60.4 (DOUT)
- net at LED59.2 (DIN): now also LED60.4 (DOUT); no longer LED58.4 (DOUT)
- net at LED59.4 (DOUT): now also LED58.2 (DIN); no longer LED60.2 (DIN)
- net at LED65.2 (DIN): now also LED66.4 (DOUT); no longer LED64.4 (DOUT)
- net at LED46.2 (DIN): now also LED47.4 (DOUT); no longer LED45.4 (DOUT)
- net at LED78.4 (DOUT): now also LED77.2 (DIN); no longer LED79.2 (DIN)
- net at LED80.2 (DIN): no longer LED79.4 (DOUT)
- net at LED21.4 (DOUT): now also LED20.2 (DIN); no longer LED22.2 (DIN)
- net at LED11.2 (DIN): now also LED12.4 (DOUT); no longer LED10.4 (DOUT)
- net at LED11.4 (DOUT): now also LED10.2 (DIN); no longer LED12.2 (DIN)
- net at LED55.4 (DOUT): now also LED54.2 (DIN); no longer LED56.2 (DIN)
- net at LED9.4 (DOUT): now also LED8.2 (DIN); no longer LED10.2 (DIN)
- net at LED80.4 (DOUT): now also LED79.2 (DIN)
- new net: LED25.2 (DIN), LED26.4 (DOUT)
- new net: LED36.2 (DIN), LED37.4 (DOUT)
- new net: LED15.2 (DIN), LED16.4 (DOUT)
- new net: LED70.2 (DIN), LED71.4 (DOUT)
- new net: LED1.2 (DIN), LED2.4 (DOUT)
- new net: LED51.2 (DIN), LED52.4 (DOUT)
- new net: LED22.2 (DIN), LED23.4 (DOUT)
- new net: LED33.2 (DIN), LED34.4 (DOUT)
- new net: LED12.2 (DIN), LED13.4 (DOUT)

Commit message: Created BOM and added parts. Created v0.1 prototype 2x2
Parts:
- LED1, LED10, LED11, LED12, LED13, LED14, LED15, LED16, LED17, LED18, LED19, LED2, LED20, LED21, LED22, LED23, LED24, LED25, LED26, LED27, LED28, LED29, LED3, LED30, LED31, LED32, LED33, LED34, LED35, LED36, LED37, LED38, LED39, LED4, LED40, LED41, LED42, LED43, LED44, LED45, LED46, LED47, LED48, LED49, LED5, LED50, LED51, LED52, LED53, LED54, LED55, LED56, LED57, LED58, LED59, LED6, LED60, LED61, LED62, LED63, LED64, LED65, LED66, LED67, LED68, LED69, LED7, LED70, LED71, LED72, LED73, LED74, LED75, LED76, LED77, LED78, LED79, LED8, LED80, LED9: footprint LED_SMD:LED_SK6812_PLCC4_5.0x5.0mm_P3.2mm -> BOM:LED_SK6812_PLCC4_5.0x5.0mm_P1.6mm
