File: Prototype/Prototype.kicad_pcb (KiCad board)
At the start: 4 copper layers, 52 x 42.3 mm, 17 parts, among them J1 Conn_01x07_Socket, SW82 SW_Push, SW84 SW_Push, SW86 SW_Push, SW87 SW_Push

Commit message: work on v0.3 of prototype board, new mounting holes/trace runs
Parts:
- removed D82, D84, D86, D87: D, BOM:CR_48W-E3-08_VIS
- removed SW82, SW84, SW86, SW87: SW_Push, ScottoKeebs_Hotswap:Hotswap_MX_1.00u
- added D1: D, Diode_SMD:D_SOD-323, B.Cu at (-69.8, -28.6)
- added D2: D, Diode_SMD:D_SOD-323, B.Cu at (-50.7, -28.7)
- added D3: D, Diode_SMD:D_SOD-323, B.Cu at (-31.7, -28.6)
- added D4: D, Diode_SMD:D_SOD-323, B.Cu at (-12.7, -28.6)
- added D5: D, Diode_SMD:D_SOD-323, B.Cu at (-69.8, -9.50)
- added D6: D, Diode_SMD:D_SOD-323, B.Cu at (-50.7, -9.40)
- added D7: D, Diode_SMD:D_SOD-323, B.Cu at (-31.8, -9.56)
- added D8: D, Diode_SMD:D_SOD-323, B.Cu at (-12.7, -9.49)
- added J2: Conn_01x04, Connector_PinSocket_2.00mm:PinSocket_1x04_P2.00mm_Vertical, B.Cu at (-41.1, -1.20)
- added J3: Conn_01x06, Connector_PinSocket_2.00mm:PinSocket_1x06_P2.00mm_Horizontal, B.Cu at (-74.9, -13.9)
- added J4: Conn_01x04, Connector_PinSocket_2.00mm:PinSocket_1x04_P2.00mm_Vertical, B.Cu at (-37.0, -27.9)
- added SW1: SW_Push, ScottoKeebs_Hotswap:Hotswap_MX_1.00u, F.Cu at (-66.7, -28.6)
- added SW2: SW_Push, ScottoKeebs_Hotswap:Hotswap_MX_1.00u, F.Cu at (-47.6, -28.6)
- added SW3: SW_Push, ScottoKeebs_Hotswap:Hotswap_MX_1.00u, F.Cu at (-28.6, -28.6)
- added SW4: SW_Push, ScottoKeebs_Hotswap:Hotswap_MX_1.00u, F.Cu at (-9.53, -28.6)
- added SW5: SW_Push, ScottoKeebs_Hotswap:Hotswap_MX_1.00u, F.Cu at (-66.7, -9.53)
- added SW6: SW_Push, ScottoKeebs_Hotswap:Hotswap_MX_1.00u, F.Cu at (-47.6, -9.53)
- added SW7: SW_Push, ScottoKeebs_Hotswap:Hotswap_MX_1.00u, F.Cu at (-28.6, -9.53)
- added SW8: SW_Push, ScottoKeebs_Hotswap:Hotswap_MX_1.00u, F.Cu at (-9.53, -9.53)
- C1, C2, C3, C4: footprint BOM:CAPC1608X87N -> Capacitor_SMD:C_0402_1005Metric
- J1: value Conn_01x07_Socket -> Conn_01x04; footprint Connector_PinSocket_1.00mm:PinSocket_1x07_P1.00mm_Vertical -> Connector_PinSocket_2.00mm:PinSocket_1x04_P2.00mm_Vertical; moved to B.Cu
- moved J1 208.9 mm to (-41.1, -36.9), turned to -90 degrees
- moved C2 206.4 mm to (-51.1, -33.9), turned to 90 degrees
- moved LED1 198.8 mm to (-66.7, -34.7), turned to 90 degrees
- moved LED2 198.8 mm to (-47.6, -34.7), turned to 90 degrees
- moved C1 196.5 mm to (-70.2, -33.9), turned to 90 degrees
- moved LED3 178.2 mm to (-66.7, -15.7), turned to -90 degrees
- moved C3 177.5 mm to (-63.3, -17.8), turned to -90 degrees
- moved LED4 164.5 mm to (-47.6, -15.8), turned to -90 degrees
- moved C4 161.1 mm to (-44.2, -17.8), turned to -90 degrees
Connections:
- J1 pad 1: +5V -> C1
- J1 pad 2: GND -> C2
- J1 pad 3: C1 -> C3
- J1 pad 4: C2 -> C4
- LED1 pad 2: Net-(LED1-DIN) -> RGBW_DATA_IN
- LED2 pad 2: RGBW_DATA -> Net-(LED1-DOUT)
- LED2 pad 4: Net-(LED1-DIN) -> RGBW_DATA_OUT
- LED3 pad 2: Net-(LED1-DOUT) -> Net-(LED3-DIN)
- LED3 pad 4: Net-(LED3-DOUT) -> RGBW_DATA_JUMPER_OUT
- LED4 pad 2: Net-(LED3-DOUT) -> RGBW_DATA_JUMPER_IN
- LED4 pad 4: unconnected-(LED4-DOUT-Pad4) -> Net-(LED3-DIN)
Routing:
- net R1: track 0.00 -> 86.4 mm, vias 0 -> 4
- net C1: track 19.4 -> 95.4 mm
- net C4: track 0.00 -> 72.2 mm
- net R2: track 0.00 -> 72.1 mm, vias 0 -> 4
- net C2: track 19.4 -> 63.0 mm
- net C3: track 0.00 -> 39.0 mm
- net RGBW_DATA_IN: track 0.00 -> 23.2 mm
- net RGBW_DATA: track 20.4 -> 0.00 mm
- net RGBW_DATA_JUMPER_IN: track 0.00 -> 20.2 mm, vias 0 -> 1
- net Net-(LED1-DIN): track 19.7 -> 0.00 mm
- net Net-(LED1-DOUT): track 0.00 -> 19.0 mm
- net GND: track 7.91 -> 26.8 mm
- net Net-(LED3-DIN): track 0.00 -> 17.9 mm
- net +5V: track 109.5 -> 93.9 mm, vias 2 -> 4
- net Net-(D4-A): track 0.00 -> 12.7 mm
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- added copper zone on In2.Cu, net GND
Other:
- board size 52 x 42.3 mm -> 85.2 x 38.1 mm
